File: power_dbg.kicad_sch (KiCad schematic)
At the start: 13 parts, among them J2 Conn_01x02, J3 Conn_ARM_JTAG_SWD_10, J6 USB_C_Receptacle_USB2.0, U2 AMS1117-33, U3 SRV05-4

Commit message: update to match library changes, update to include repo
After moving all in house, label the board with a correct internal url
Updated the library to have new "LCSC Part #" instead of "LCSC Part#"
and updated all symbols to match that.  Updated to the neweer standard
14/16 pin usb connector symbols

_should_ be final for gerbesr
Parts:
- removed J6: USB_C_Receptacle_USB2.0, Connector_USB:USB_C_Receptacle_GCT_USB4105-xx-A_16P_TopMnt_Horizontal, symbol Connector:USB_C_Receptacle_USB2.0
- added J6: USB_C_Receptacle_USB2.0_16P, symbol Connector:USB_C_Receptacle_USB2.0_16P
- C4, C5: LCSC Part # (none) -> C15850
- R11: LCSC Part # (none) -> C21189
- R7, R8: LCSC Part # (none) -> C23186
- U3: LCSC Part # (none) -> C7420376; MPN SRV05-4 -> SRV05-4
Connections:
- net +5V: now also J6.A4 (VBUS), J6.A9 (VBUS), J6.B4 (VBUS), J6.B9 (VBUS)
- net GND: now also J6.A1 (GND), J6.A12 (GND), J6.B1 (GND), J6.B12 (GND), J6.S1 (SHIELD)
- net USBN: now also J6.A7 (D-), J6.B7 (D-)
- net USBP: now also J6.A6 (D+), J6.B6 (D+)
- net at R7.1: now also J6.A5 (CC1)
- net at R8.1: now also J6.B5 (CC2)

Commit message: resynced to pcb to get symbol updates
found out that the production files didn't have the right symbol updates
for the jlc data, so resynced all again
Parts:
- J6: footprint (none) -> Connector_USB:USB_C_Receptacle_GCT_USB4105-xx-A_16P_TopMnt_Horizontal
Changed lines of the file:
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@@
 			)
 		)
-		(property "Footprint" ""
+		(property "Footprint" "Connector_USB:USB_C_Receptacle_GCT_USB4105-xx-A_16P_TopMnt_Horizontal"
 			(at 161.29 88.9 0)
 			(effects

Commit message: yet more part number syncing
Because parts go to pcb as well, lots more syncing ws needed. hopefully
this will be more streamlined in future
Parts:
- J2: LCSC Part # (none) -> C430323
- J3: LCSC Part # (none) -> C6332249
- J6: LCSC Part # (none) -> C2927038
- U2: LCSC Part # (none) -> C6186
Changed lines of the file:
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@@
+			)
+		)
+		(property "LCSC Part #" "C6332249"
+			(at 96.52 160.02 0)
+			(effects
+				(font
+					(size 1.27 1.27)
+				)
+				(hide yes)
 			)
 		)
@@
 			)
 		)
+		(property "LCSC Part #" "C430323"
+			(at 58.42 96.52 0)
+			(effects
+				(font
+					(size 1.27 1.27)
+				)
+				(hide yes)
+			)
+		)
 		(pin "2"
 		)
@@
 			)
 		)
+		(property "LCSC Part #" "C6186"
+			(at 63.5 58.42 0)
+			(effects
+				(font
+					(size 1.27 1.27)
+				)
+				(hide yes)
+			)
+		)
 		(pin "1"
 		)
@@
 			(at 157.48 88.9 0)
 			(effects
+				(font
+					(size 1.27 1.27)
+				)
+				(hide yes)
+			)
+		)
+		(property "LCSC Part #" "C2927038"
+			(at 157.48 88.9 0)
+			(effects
