File: hw/bonus_io.kicad_sch (KiCad schematic)
At the start: 7 parts, among them J10 Conn_01x03, J7 Conn_01x03, J8 Conn_01x03, J9 Conn_01x03, M7 Servo_x5, U5 ULN2003A

Commit message: drop the old lcsc part#
keep just the "LCSC Part #" that the plugin wants, drop the "LCSC Part#"
Parts:
- C12: LCSC Part# C14663 -> (none)
- J10, J7, J8, J9: LCSC Part# C8406 -> (none)
- M7: LCSC Part# C32713292 -> (none)
- U5: LCSC Part# C7512 -> (none)
Changed lines of the file:
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@@
-			)
-		)
-		(property "LCSC Part#" "C8406"
-			(at 243.84 139.7 0)
-			(effects
-				(font
-					(size 1.27 1.27)
-				)
-				(hide yes)
 			)
 		)
@@
 			)
 		)
-		(property "LCSC Part#" "C8406"
-			(at 243.84 127 0)
-			(effects
-				(font
-					(size 1.27 1.27)
-				)
-				(hide yes)
-			)
-		)
 		(property "MPN" "WJ15EDGRC-3.81-3P"
 			(at 243.84 127 0)
@@
 			)
 		)
-		(property "LCSC Part#" "C8406"
-			(at 243.84 154.94 0)
-			(effects
-				(font
-					(size 1.27 1.27)
-				)
-				(hide yes)
-			)
-		)
 		(property "MPN" "WJ15EDGRC-3.81-3P"
 			(at 243.84 154.94 0)
@@
 		)
 		(property "Description" "Generic connector, single row, 01x03, script generated (kicad-library-utils/schlib/autogen/connector/)"
-			(at 243.84 114.3 0)
-			(effects
-				(font
-					(size 1.27 1.27)
-				)
-				(hide yes)
-			)
-		)
-		(property "LCSC Part#" "C8406"
 			(at 243.84 114.3 0)
 			(effects
@@
 			)
 		)
-		(property "LCSC Part#" "C14663"
-			(at 213.36 110.49 0)
-			(effects
-				(font
-					(size 1.27 1.27)
-				)
-				(hide yes)
-			)
-		)
 		(property "LCSC Part #" "C14663"
 			(at 213.36 110.49 0)
@@
 			)
 		)
-		(property "LCSC Part#" "C7512"
-			(at 195.58 124.46 0)
-			(effects
-				(font
-					(size 1.27 1.27)
-				)
-				(hide yes)
-			)
-		)
 		(property "LCSC Part #" "C7512"
 			(at 195.58 124.46 0)
@@
 			(effects
 				(font
-					(size 1.27 1.27)
-				)
-				(hide yes)
-			)
-		)
-		(property "LCSC Part#" "C32713292"
-			(at 76.454 65.024 0)
-			(effects
-				(font
