File: hw/bridge_sim.kicad_sch (KiCad schematic)
At the start: 21 parts, among them J1 Conn_01x06, J5 Conn_01x06, Q1 AO3400A, U1 MCP4131-104E/SN, U4 MCP4131-104E/SN, U7 LTV-817S

Commit message: drop the old lcsc part#
keep just the "LCSC Part #" that the plugin wants, drop the "LCSC Part#"
Parts:
- C2: LCSC Part# C14663 -> (none)
- J1: LCSC Part# C387811 -> (none)
- Q1: LCSC Part# C20917 -> (none)
- R1, R18: LCSC Part# C23138 -> (none)
- R10, R16, R17: LCSC Part# C21189 -> (none)
- R14, R5: LCSC Part# C17633 -> (none)
- R15: LCSC Part# C17470 -> (none)
- R2, R23, R3, R4: LCSC Part# C17630 -> (none)
- R21: LCSC Part# C4216 -> (none)
- R6: LCSC Part# C17556 -> (none)
- U1, U4: LCSC Part# C636034 -> (none)
- U7: LCSC Part# C106900 -> (none)
Changed lines of the file:
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@@
-			)
-		)
-		(property "LCSC Part#" "C106900"
-			(at 104.14 35.56 0)
-			(effects
-				(font
-					(size 1.27 1.27)
-				)
-				(hide yes)
 			)
 		)
@@
 			)
 		)
-		(property "LCSC Part#" "C17630"
-			(at 175.26 93.98 0)
-			(effects
-				(font
-					(size 1.27 1.27)
-				)
-				(hide yes)
-			)
-		)
 		(property "LCSC Part #" "C17630"
 			(at 175.26 93.98 0)
@@
 			)
 		)
-		(property "LCSC Part#" "C17633"
-			(at 208.28 93.98 0)
-			(effects
-				(font
-					(size 1.27 1.27)
-				)
-				(hide yes)
-			)
-		)
 		(property "LCSC Part #" "C17633"
 			(at 208.28 93.98 0)
@@
 			)
 		)
-		(property "LCSC Part#" "C4216"
-			(at 124.46 33.02 0)
-			(effects
-				(font
-					(size 1.27 1.27)
-				)
-				(hide yes)
-			)
-		)
 		(property "LCSC Part #" "C4216"
 			(at 124.46 33.02 0)
@@
 			)
 		)
-		(property "LCSC Part#" "C17633"
-			(at 165.1 86.36 0)
-			(effects
-				(font
-					(size 1.27 1.27)
-				)
-				(hide yes)
-			)
-		)
 		(property "LCSC Part #" "C17633"
 			(at 165.1 86.36 0)
@@
 			)
 		)
-		(property "LCSC Part#" "C20917"
-			(at 137.16 38.1 0)
-			(effects
-				(font
-					(size 1.27 1.27)
-				)
-				(hide yes)
-			)
-		)
 		(property "jlcbasic" "basic"
 			(at 137.16 38.1 0)
@@
 			)
 		)
-		(property "LCSC Part#" "C636034"
-			(at 71.12 86.36 0)
-			(effects
-				(font
-					(size 1.27 1.27)
-				)
-				(hide yes)
-			)
-		)
 		(property "LCSC Part #" "C636034"
 			(at 71.12 86.36 0)
@@
 			)
 		)
-		(property "LCSC Part#" "C17630"
-			(at 175.26 81.28 0)
-			(effects
-				(font
-					(size 1.27 1.27)
-				)
-				(hide yes)
-			)
-		)
 		(property "LCSC Part #" "C17630"
 			(at 175.26 81.28 0)
@@
 			)
 		)
-		(property "LCSC Part#" "C21189"
-			(at 147.32 86.36 0)
-			(effects
-				(font
-					(size 1.27 1.27)
-				)
-				(hide yes)
-			)
-		)
 		(property "MPN" "0603WAF0000T5E"
 			(at 147.32 86.36 0)
@@
 			)
 		)
-		(property "LCSC Part#" "C17470"
-			(at 101.6 114.3 0)
-			(effects
-				(font
-					(size 1.27 1.27)
-				)
-				(hide yes)
-			)
-		)
 		(property "LCSC Part #" "C17470"
 			(at 101.6 114.3 0)
@@
 			)
 		)
-		(property "LCSC Part#" "C14663"
-			(at 55.88 113.03 0)
-			(effects
-				(font
-					(size 1.27 1.27)
-				)
-				(hide yes)
-			)
-		)
 		(property "LCSC Part #" "C14663"
 			(at 55.88 113.03 0)
@@
 			)
 		)
-		(property "LCSC Part#" "C21189"
-			(at 152.4 81.28 0)
-			(effects
-				(font
-					(size 1.27 1.27)
-				)
-				(hide yes)
-			)
-		)
 		(property "MPN" "0603WAF0000T5E"
 			(at 152.4 81.28 0)
@@
 			)
 		)
-		(property "LCSC Part#" "C17630"
-			(at 200.66 81.28 0)
-			(effects
-				(font
-					(size 1.27 1.27)
-				)
-				(hide yes)
-			)
-		)
 		(property "LCSC Part #" "C17630"
 			(at 200.66 81.28 0)
@@
 			)
 		)
-		(property "LCSC Part#" "C17630"
-			(at 200.66 93.98 0)
-			(effects
-				(font
-					(size 1.27 1.27)
-				)
-				(hide yes)
-			)
-		)
 		(property "LCSC Part #" "C17630"
 			(at 200.66 93.98 0)
@@
 		)
 		(property "MPN" "0603WAF3300T5E"
-			(at 124.46 43.18 0)
-			(effects
-				(font
-					(size 1.27 1.27)
-				)
-				(hide yes)
-			)
-		)
-		(property "LCSC Part#" "C23138"
 			(at 124.46 43.18 0)
 			(effects
@@
 			)
 		)
-		(property "LCSC Part#" "C23138"
-			(at 81.28 33.02 0)
-			(effects
-				(font
-					(size 1.27 1.27)
-				)
-				(hide yes)
-			)
-		)
 		(property "LCSC Part #" "C23138"
 			(at 81.28 33.02 0)
@@
 			)
 		)
-		(property "LCSC Part#" "C636034"
-			(at 71.12 134.62 0)
-			(effects
-				(font
-					(size 1.27 1.27)
-				)
-				(hide yes)
-			)
-		)
 		(property "LCSC Part #" "C636034"
 			(at 71.12 134.62 0)
@@
 			)
 		)
-		(property "LCSC Part#" "C387811"
-			(at 228.6 35.56 0)
-			(effects
-				(font
-					(size 1.27 1.27)
-				)
-				(hide yes)
-			)
-		)
 		(property "LCSC Part #" "C387811"
 			(at 228.6 35.56 0)
@@
 			)
 		)
-		(property "LCSC Part#" "C21189"
-			(at 101.6 93.98 0)
-			(effects
-				(font
-					(size 1.27 1.27)
-				)
-				(hide yes)
-			)
-		)
 		(property "MPN" "0603WAF0000T5E"
 			(at 101.6 93.98 0)
@@
 			(at 215.9 93.98 0)
 			(effects
-				(font
-					(size 1.27 1.27)
-				)
-				(hide yes)
-			)
-		)
-		(property "LCSC Part#" "C17556"
-			(at 215.9 93.98 0)
-			(effects
