File: hw/kcell-faker.kicad_sch (KiCad schematic)
At the start: 27 parts, among them J4 DBG, SW1 BOOT, SW2 RST, SW3 UP, SW4 DOWN, SW5 RANGE, U6 ESP32-S3-MINI-1

Commit message: drop the old lcsc part#
keep just the "LCSC Part #" that the plugin wants, drop the "LCSC Part#"
Parts:
- C1, C3: LCSC Part# C15850 -> (none)
- C10, C11, C14, C6, C7, C8: LCSC Part# C14663 -> (none)
- C9: LCSC Part# C15849 -> (none)
- D1: LCSC Part# C84256 -> (none)
- D3: LCSC Part# C2297 -> (none)
- J4: LCSC Part# C2937625 -> (none)
- R12, R13: LCSC Part# C23138 -> (none)
- R19: LCSC Part# C23193 -> (none)
- R20, R22: LCSC Part# C25804 -> (none)
- R9: LCSC Part# C25804 -> (none); jlc-basic 1 -> (none)
- SW1, SW2, SW3, SW4, SW5: LCSC Part# C318884 -> (none); jlc-basic 1 -> (none)
- U6: LCSC Part# C2913206 -> (none)
