File: hw/power_dbg.kicad_sch (KiCad schematic)
At the start: 13 parts, among them J2 Conn_01x02, J3 Conn_ARM_JTAG_SWD_10, J6 USB_C_Receptacle_USB2.0_16P, U2 AMS1117-33, U3 SRV05-4

Commit message: drop the old lcsc part#
keep just the "LCSC Part #" that the plugin wants, drop the "LCSC Part#"
Parts:
- C4, C5: LCSC Part# C15850 -> (none)
- J2: LCSC Part# C430323 -> (none)
- J3: LCSC Part# C6332249 -> (none)
- J6: LCSC Part# C2927038 -> (none)
- R11: LCSC Part# C21189 -> (none)
- R7, R8: LCSC Part# C23186 -> (none)
- U2: LCSC Part# C6186 -> (none); jlc-basic 1 -> (none)
- U3: LCSC Part# C7420376 -> (none); jlc-basic 1 -> (none)
Changed lines of the file:
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@@
-			)
-		)
-		(property "LCSC Part#" "C15850"
-			(at 76.2 67.31 0)
-			(effects
-				(font
-					(size 1.27 1.27)
-				)
-				(hide yes)
 			)
 		)
@@
 			)
 		)
-		(property "LCSC Part#" "C6332249"
-			(at 96.52 160.02 0)
-			(effects
-				(font
-					(size 1.27 1.27)
-				)
-				(hide yes)
-			)
-		)
 		(property "LCSC Part #" "C6332249"
 			(at 96.52 160.02 0)
@@
 			)
 		)
-		(property "LCSC Part#" "C430323"
-			(at 58.42 96.52 0)
-			(effects
-				(font
-					(size 1.27 1.27)
-				)
-				(hide yes)
-			)
-		)
 		(property "LCSC Part #" "C430323"
 			(at 58.42 96.52 0)
@@
 			)
 		)
-		(property "LCSC Part#" "C21189"
-			(at 116.84 152.4 0)
-			(effects
-				(font
-					(size 1.27 1.27)
-				)
-				(hide yes)
-			)
-		)
 		(property "MPN" "0603WAF0000T5E"
 			(at 116.84 152.4 0)
@@
 			)
 		)
-		(property "LCSC Part#" "C23186"
-			(at 195.58 78.74 0)
-			(effects
-				(font
-					(size 1.27 1.27)
-				)
-				(hide yes)
-			)
-		)
 		(property "LCSC Part #" "C23186"
 			(at 195.58 78.74 0)
@@
 			)
 		)
-		(property "LCSC Part#" "C23186"
-			(at 195.58 81.28 0)
-			(effects
-				(font
-					(size 1.27 1.27)
-				)
-				(hide yes)
-			)
-		)
 		(property "LCSC Part #" "C23186"
 			(at 195.58 81.28 0)
@@
 			)
 		)
-		(property "jlc-basic" "1"
-			(at 220.98 91.44 0)
-			(effects
-				(font
-					(size 1.27 1.27)
-				)
-				(hide yes)
-			)
-		)
 		(property "lcsc2#" "C85364"
 			(at 220.98 91.44 0)
@@
 		(property "MPN" "SRV05-4"
 			(at 224.0981 76.2 0)
-			(effects
-				(font
-					(size 1.27 1.27)
-				)
-				(justify right)
-			)
-		)
-		(property "LCSC Part#" "C7420376"
-			(at 224.0981 78.74 0)
 			(effects
 				(font
@@
 			)
 		)
-		(property "jlc-basic" "1"
-			(at 63.5 58.42 0)
-			(effects
-				(font
-					(size 1.27 1.27)
-				)
-				(hide yes)
-			)
-		)
 		(property "jlcbasic" "basic"
-			(at 63.5 58.42 0)
-			(effects
-				(font
-					(size 1.27 1.27)
-				)
-				(hide yes)
-			)
-		)
-		(property "LCSC Part#" "C6186"
 			(at 63.5 58.42 0)
 			(effects
@@
 			)
 		)
-		(property "LCSC Part#" "C2927038"
-			(at 157.48 88.9 0)
-			(effects
-				(font
-					(size 1.27 1.27)
-				)
-				(hide yes)
-			)
-		)
 		(property "MPN" "USB-TYPE-C-018"
 			(at 157.48 88.9 0)
@@
 			(effects
 				(font
-					(size 1.27 1.27)
-				)
-				(hide yes)
-			)
-		)
-		(property "LCSC Part#" "C15850"
-			(at 50.8 67.31 0)
-			(effects
-				(font
